File: gt-jtx/hardware/gt-jtx.brd (EAGLE design)
At the start: 100 x 80 mm, 6 parts, among them IC1 MEGA8-P

Commit message: gt-jtx now has a board layout and a schematic.
git-svn-id: https://gt-jtx.googlecode.com/svn/trunk@15 79910f2a-facc-22ab-b1ea-80da55196309
Parts:
- removed JP2: (no value), pinhead:1X10
- removed JP3: (no value), pinhead:1X03
- removed JP4: (no value), pinhead:1X02
- removed LD1: (no value), led:DUOLED-C-5MM
- added ACT: (no value), led:DUOLED-C-5MM
- added INPUT, LCD: (no value), pinhead:1X10
- added POWER: (no value), pinhead:1X02
- added PPM: (no value), pinhead:1X03
- added R1: (no value), pot:CA6V
- JP1: device pinhead:1X10 -> pinhead:1X06
- moved JP1 10.5 mm to (14.0, 66.0)
- moved IC1 8.03 mm to (24.1, 57.1)
Connections:
- new net N$10: IC1.27, JP1.2
- new net N$11: IC1.28, JP1.1
- new net N$12: IC1.19, LCD.10
- new net N$13: IC1.18, LCD.9
- new net N$14: IC1.17, LCD.8
- new net N$15: IC1.16, LCD.7
- new net N$16: ACT.AX, IC1.15, PPM.1
- new net N$17: IC1.3, INPUT.7
- new net N$18: IC1.4, INPUT.6
- new net N$19: IC1.5, INPUT.5
- new net N$20: IC1.6, INPUT.4
- new net N$21: IC1.11, INPUT.3
- new net N$22: IC1.13, INPUT.1
- new net N$23: IC1.12, INPUT.2
- new net N$9: LCD.3, R1.S
- net +5V: now also ACT.AR, IC1.21, INPUT.10, LCD.1, POWER.1, PPM.3, R1.A; no longer JP1.2, JP2.10, JP3.3, JP4.1, LD1.AX
- net GND: now also ACT.C, INPUT.9, LCD.2, POWER.2, PPM.2, R1.E; no longer JP1.1, JP2.9, JP3.2, JP4.2, LD1.C
- net N$1: now also JP1.6; no longer JP2.8
- net N$2: now also JP1.5; no longer JP2.7
- net N$3: now also JP1.4; no longer JP2.6
- net N$4: now also JP1.3; no longer JP2.5
- net N$5: now also LCD.4; no longer JP1.3
- net N$6: now also LCD.5; no longer JP1.4
- net N$7: now also LCD.6; no longer JP1.5
- net N$8: now also IC1.2, INPUT.8; no longer IC1.15, JP3.1, LD1.AR
Routing:
- net N$24: track 0.00 -> 177.8 mm
- net N$16: track 0.00 -> 62.6 mm
- net GND: track 101.4 -> 151.8 mm
- net N$5: track 42.3 -> 7.93 mm
- net N$9: track 0.00 -> 33.9 mm
- net N$23: track 0.00 -> 26.0 mm
- net N$12: track 0.00 -> 21.2 mm
- net N$13: track 0.00 -> 17.7 mm
- net +5V: track 119.9 -> 136.9 mm
- net N$14: track 0.00 -> 14.1 mm
- net N$21: track 0.00 -> 12.3 mm
- net N$22: track 0.00 -> 12.3 mm
- net N$15: track 0.00 -> 10.5 mm
- net N$6: track 29.3 -> 19.1 mm
- net N$8: track 15.1 -> 5.08 mm
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Other:
- board text added: "+ PWR"
- board text added: "CONT"
- board text added: "INPUTA"
- board text added: "INPUTB"
- board text added: "LCD"
- board text added: "PPM"
- board text added: "ver 1.0"
