File: gt-jtx/hardware/gt-jtx-m16-ver1.0.brd (EAGLE design)
At the start: 100 x 80 mm, 11 parts, among them IC1 MEGA16-P

Commit message: git-svn-id: https://gt-jtx.googlecode.com/svn/trunk@43 79910f2a-facc-22ab-b1ea-80da55196309
Parts:
- renumbered INPUT to TRIMS, INPUT1 to ANALOG, INPUT2 to DIGITAL, JP1 to ISP, LED1 to LED, POWER to PWR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
Other:
- board text added: "m16"
- board text added: "ver 1.0"
- board text removed: "ver 2.0"
