File: hardware/gt-jtx-m32-ver1.0.brd (EAGLE design)
At the start: 100 x 80 mm, 11 parts, among them IC1 MEGA32-P

Commit message: added speaker and switch ports changed ppm pin to PD5
git-svn-id: https://gt-jtx.googlecode.com/svn/trunk@69 79910f2a-facc-22ab-b1ea-80da55196309
Parts:
- added SPK_SW: (no value), pinhead:1X03
- moved PPM 9.25 mm to (21.6, 35.6)
Connections:
- removed net GND: ANALOG.1, IC1.11, IC1.31, LCD_CTRL.9, LCD_DATA.9, LED.K, PPM.2, PWR.2, TRIMS.1, VR1.E
- new net N$5: IC1.20, SPK_SW.1
- new net N$6: IC1.21, SPK_SW.3
- new net SPK_SW: ANALOG.1, IC1.11, IC1.31, LCD_CTRL.9, LCD_DATA.9, LED.K, PPM.2, PWR.2, SPK_SW.2, TRIMS.1, VR1.E
- net N$15: now also IC1.19; no longer IC1.21
Routing:
- net GND: track 142.3 -> 0.00 mm
- net SPK_SW: track 0.00 -> 134.9 mm
- net +5V: track 217.9 -> 228.9 mm
- net N$6: track 0.00 -> 8.45 mm
- net N$15: track 7.40 -> 15.1 mm
- net N$5: track 0.00 -> 6.66 mm
- added copper zone on layer 1, net SPK_SW
- removed copper zone on layer 1, net GND
Other:
- board text added: "m32"
- board text removed: "m16"

Commit message: fixed some of the hardware design
git-svn-id: https://gt-jtx.googlecode.com/svn/trunk@70 79910f2a-facc-22ab-b1ea-80da55196309
Parts:
- moved LED 42.2 mm to (35.6, 63.5)
- moved PPM 21.6 mm to (22.9, 57.1), turned to 90 degrees
- moved PWR 13.7 mm to (57.1, 66.0), turned to 0 degrees
- moved R2 10.2 mm to (57.1, 55.9)
- moved VR1 10.2 mm to (45.7, 63.5)
- moved SPK_SW 2.54 mm to (22.9, 35.6)
- moved IC1 1.27 mm to (54.6, 35.6)
- moved ISP 1.27 mm to (59.7, 61.0), turned to 180 degrees
Connections:
- removed net N$33: IC1.6, ISP.6, TRIMS.5
- removed net N$34: IC1.7, ISP.5, TRIMS.4
- removed net RST: IC1.9, ISP.1, LCD_CTRL.1, R2.2
- removed net SPK_SW: ANALOG.1, IC1.11, IC1.31, LCD_CTRL.9, LCD_DATA.9, LED.K, PPM.2, PWR.2, SPK_SW.2, TRIMS.1, VR1.E
- new net GND: ANALOG.1, IC1.11, IC1.31, ISP.1, LCD_CTRL.2, LCD_DATA.9, LED.K, PPM.2, PWR.2, SPK_SW.2, TRIMS.2, VR1.E
- new net N$12: IC1.6, ISP.6
- new net N$13: IC1.7, ISP.2
- new net N$14: IC1.8, ISP.3
- new net N$9: IC1.9, ISP.4, LCD_CTRL.10, R2.2
- net +5V: now also ISP.5, LCD_CTRL.1, TRIMS.1; no longer ISP.3, LCD_CTRL.10, TRIMS.2
- net CONTRA_ADJ: now also LCD_CTRL.3; no longer LCD_CTRL.2
- net N$28: no longer IC1.8, ISP.4
Routing:
- net GND: track 0.00 -> 244.0 mm
- net SPK_SW: track 134.9 -> 0.00 mm
- net N$28: track 74.4 -> 0.00 mm
- net N$34: track 63.9 -> 0.00 mm
- net N$12: track 0.00 -> 62.9 mm
- net RST: track 54.8 -> 0.00 mm
- net +5V: track 228.9 -> 180.3 mm
- net N$33: track 42.0 -> 0.00 mm
- net N$9: track 0.00 -> 38.0 mm
- net N$13: track 0.00 -> 26.0 mm
- net N$14: track 0.00 -> 18.8 mm
- net CONTRA_ADJ: track 14.3 -> 22.0 mm
- net N$15: track 15.1 -> 19.4 mm
- net N$5: track 6.66 -> 9.72 mm
- net RW: track 8.89 -> 7.62 mm
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- added copper zone on layer 1, net GND
- removed copper zone on layer 1, net SPK_SW
